Commit message: Updated arduino bot URDF file

File: src/arduinobot_description/urdf/arduinobot.urdf.xacro (robot description, xacro)
@@ -37,7 +37,15 @@
         <material name="PureBlack">
         <color rgba="1.0 1.0 1.0 1.0"/>
-  <!-- Pure black, fully opaque -->
     </material>
     </visual>
+    <collision>
+      <origin rpy="0 0 0" xyz="0.04 -0.04  0.15"/>
+      <geometry>
+        <mesh filename="package://arduinobot_description/meshes/base_plate1.stl" scale="0.01 0.01 0.01"/>
+      </geometry>
+        <material name="PureBlack">
+        <color rgba="1.0 1.0 1.0 1.0"/>
+    </material>
+    </collision>
   </link>
   <!-- Revolute Joint: base_link -> base_plate -->

Commit message: updated at 21/08/2025

File: src/arduinobot_description/urdf/arduinobot.urdf.xacro (robot description, xacro)
@@ -5,8 +5,17 @@
   <xacro:property name="effort" value="30.0"/>
   <xacro:property name="velocity" value="10.0"/>
+  <xacro:macro name="default_inertial" params="mass">
+         <inertial>
+      <mass value="${mass}"/>
+      <inertia ixx="1.0" ixy="0.0" ixz="0.0"
+               iyy="1.0" iyz="0.0"
+               izz="1.0"/>
+    </inertial>
+  </xacro:macro>
   <!-- Root Link -->
   <link name="world"/>
   <!-- Base Link -->
   <link name="base_link">
+   <xacro:default_inertial mass="1.0"/>
     <visual>
       <origin rpy="0 0 0" xyz="0 0 0"/>
@@ -30,4 +39,5 @@
   <!-- Base Plate Link -->
   <link name="base_plate">
+    <xacro:default_inertial mass="0.1"/>
     <visual>
       <origin rpy="0 0 0" xyz="0.04 -0.04  0.15"/>
@@ -35,7 +45,4 @@
         <mesh filename="package://arduinobot_description/meshes/base_plate1.stl" scale="0.01 0.01 0.01"/>
       </geometry>
-        <material name="PureBlack">
-        <color rgba="1.0 1.0 1.0 1.0"/>
-    </material>
     </visual>
     <collision>
@@ -44,7 +51,4 @@
         <mesh filename="package://arduinobot_description/meshes/base_plate1.stl" scale="0.01 0.01 0.01"/>
       </geometry>
-        <material name="PureBlack">
-        <color rgba="1.0 1.0 1.0 1.0"/>
-    </material>
     </collision>
   </link>
@@ -57,11 +61,18 @@
     <limit lower="${-PI/2}" upper="${PI/2}" effort="${effort}" velocity="${velocity}"/>
   </joint>
-  <link name="forword_drive" type="fixed">
+  <link name="forword_drive">
+    <xacro:default_inertial mass="0.1"/>
     <visual>
       <origin rpy="0 -${PI/2} ${PI/2}" xyz="0.20 0.075 -0.075"/>
       <geometry>
-        <mesh filename="package://arduinobot_description/meshes/forward_drive_arm.STL" scale="0.01 0.01 0.01"/>
+        <mesh filename="package://arduinobot_description/meshes/forward_drive_arm.stl" scale="0.01 0.01 0.01"/>
       </geometry>
     </visual>
+    <collision>
+      <origin rpy="0 -${PI/2} ${PI/2}" xyz="0.20 0.075 -0.075"/>
+      <geometry>
+        <mesh filename="package://arduinobot_description/meshes/forward_drive_arm.stl" scale="0.01 0.01 0.01"/>
+      </geometry>
+      </collision>
   </link>
   <joint name="joint_2" type="revolute">
@@ -72,5 +83,6 @@
     <limit lower="${-PI/2}" upper="${PI/2}" effort="${effort}" velocity="${velocity}"/>
   </joint>
-  <link name="horizontal_arm" type="revolute">
+  <link name="horizontal_arm">
+    <xacro:default_inertial mass="0.1"/>
     <visual>
       <origin rpy="0  0 1.5708 " xyz="-0.016 -0.433 -0.076"/>
@@ -79,4 +91,10 @@
       </geometry>
     </visual>
+    <collision>
+      <origin rpy="0  0 1.5708 " xyz="-0.016 -0.433 -0.076"/>
+      <geometry>
+        <mesh filename="package://arduinobot_description/meshes/horizontal_arm3.stl" scale="0.01 0.01 0.01"/>
+      </geometry>
+    </collision>
   </link>
   <joint name="joint_3" type="revolute">
@@ -87,5 +105,6 @@
     <limit lower="${-PI/2}" upper="${PI/2}" effort="${effort}" velocity="${velocity}"/>
    </joint>
-  <link name="claw_support" type="fixed">
+  <link name="claw_support">
+    <xacro:default_inertial mass="0.05"/>
     <visual>
       <origin rpy="0 0 1.5708" xyz="0.035 0.055 0.005"/>
@@ -94,4 +113,10 @@
       </geometry>
     </visual>
+    <collision>
+      <origin rpy="0 0 1.5708" xyz="0.035 0.055 0.005"/>
+      <geometry>
+        <mesh filename="package://arduinobot_description/meshes/claw_support.stl" scale="0.01 0.01 0.01"/>
+      </geometry>
+    </collision>
 </link>
   <joint name="joint_4" type="fixed">
@@ -102,5 +127,6 @@
     <limit lower="${-PI/2}" upper="${PI/2}" effort="${effort}" velocity="${velocity}"/>
   </joint>
-  <link name="griper_left" type="revolute">
+  <link name="griper_left">
+    <xacro:default_inertial mass="0.01"/>
     <visual>
       <origin rpy="0 0 4.7124" xyz="0.040 0.035 -0.08"/>
@@ -108,11 +134,14 @@
         <mesh filename="package://arduinobot_description/meshes/left_finger.stl" scale="0.01 0.01 0.01"/>
       </geometry>
-      <material name="PureBlack">
-          <color rgba="1.0 1.0 1.0 1.0"/>
-  <!-- Pure black, fully opaque -->
-     </material>
     </visual>
+    <collision>
+      <origin rpy="0 0 4.7124" xyz="0.040 0.035 -0.08"/>
+      <geometry>
+        <mesh filename="package://arduinobot_description/meshes/left_finger.stl" scale="0.01 0.01 0.01"/>
+      </geometry>
+    </collision>
   </link>
-  <link name="griper_right" type="revolute">
+  <link name="griper_right">
+    <xacro:default_inertial mass="0.01"/>
     <visual>
       <origin rpy="0 0 4.7124" xyz="-0.040 0.035 -0.08"/>
@@ -120,9 +149,11 @@
         <mesh filename="package://arduinobot_description/meshes/right_finger.stl" scale="0.01 0.01 0.01"/>
       </geometry>
-      <material name="PureBlack">
-        <color rgba="1.0 1.0 1.0 1.0"/>
-  <!-- Pure black, fully opaque -->
-    </material>
     </visual>
+    <collision>
+       <origin rpy="0 0 4.7124" xyz="-0.040 0.035 -0.08"/>
+      <geometry>
+        <mesh filename="package://arduinobot_description/meshes/right_finger.stl" scale="0.01 0.01 0.01"/>
+      </geometry>
+      </collision>
   </link>
   <joint name="joint_5" type="revolute">
